File: v_1/KiCad/latarka_1.sch (KiCad schematic (older format))
At the start: 31 parts

Commit message: latex documentation and photos
Connections:
- net PC0_RS: now reaches U?.22 ((SCL)PC0)
- net PC0_RS: now also DS?.4 (RS)
- net PC1_SW1: now reaches U?.23 ((SDA)PC1)
- net PC1_SW1: now also C?.2, R?.1, SW?.2
- net PC2_SW2: now reaches U?.24 ((TCK)PC2)
- net PC2_SW2: now also C?.2, R?.1, SW?.2
- net PC4_LED: now reaches U?.26 ((TDO)PC4)
- net PC4_LED: now also R?.2
- net PA3_encSW: now reaches U?.37 ((ADC3)PA3)
- net PA3_encSW: now also C?.2, R?.2, SW?.4
- net PA2_encB: now reaches U?.38 ((ADC2)PA2)
- net PA2_encB: now also C?.2, R?.1
- net PA1_encA: now reaches U?.39 ((ADC1)PA1)
- net PA1_encA: now also C?.1, R?.1
- net PB0_LED: no longer names the net of U?.1 ((T0/XCK)PB0)
- net PB0_LED: no longer R?.2
- removed net PB1_encSW: C?.2, R?.2, SW?.4, U?.2 ((T1)PB1)
- removed net PB2_SW1: C?.2, R?.1, SW?.2, U?.3 ((AIN0/INT2)PB2)
- removed net PB3_SW2: C?.2, R?.1, SW?.2, U?.4 ((AIN1/OC0)PB3)
- net PD0: no longer names the net of U?.14 ((RXD)PD0)
- net PD0: no longer DS?.11 (D4)
- net PD1: no longer names the net of U?.15 ((TXD)PD1)
- net PD1: no longer DS?.12 (D5)
- net PD2: no longer names the net of U?.16 ((INT0)PD2)
- net PD2: no longer DS?.13 (D6)
- net PD3 renamed PD3_ENC7
- removed net PD4_encB: C?.2, R?.1, U?.18 ((OC1B)PD4)
- removed net PD5_encA: C?.1, R?.1, U?.19 ((OC1A)PD5)
- net PD6_RS renamed PD6_ENC4
- net PD6_ENC4: now also DS?.11 (D4); no longer DS?.4 (RS)
- new net PD4_ENC6: DS?.13 (D6), U?.18 ((OC1B)PD4)
- new net PD5_ENC5: DS?.12 (D5), U?.19 ((OC1A)PD5)
Changed lines of the file:
@@
 EESchema Schematic File Version 2
 LIBS:latarka_1-rescue
-LIBS:power
-LIBS:device
-LIBS:transistors
-LIBS:conn
-LIBS:linear
-LIBS:regul
-LIBS:74xx
-LIBS:cmos4000
-LIBS:adc-dac
-LIBS:memory
-LIBS:xilinx
-LIBS:microcontrollers
-LIBS:dsp
-LIBS:microchip
-LIBS:analog_switches
-LIBS:motorola
-LIBS:texas
-LIBS:intel
-LIBS:audio
-LIBS:interface
-LIBS:digital-audio
-LIBS:philips
-LIBS:display
-LIBS:cypress
-LIBS:siliconi
-LIBS:opto
-LIBS:atmel
-LIBS:contrib
-LIBS:valves
-LIBS:pin_array_7x2
 LIBS:latarka_1-cache
 EELAYER 25 0
@@
 $EndComp
 Text GLabel 5790 2440 3    60   Input ~ 0
-PD6_RS
-Text GLabel 4040 5010 2    60   Input ~ 0
-PD6_RS
+PC0_RS
 $Comp
 L GND #PWR?
@@
 NoConn ~ 6390 2440
 Text GLabel 6490 2440 3    60   Input ~ 0
-PD0
+PD6_ENC4
 Text GLabel 6590 2440 3    60   Input ~ 0
-PD1
+PD5_ENC5
 Text GLabel 6690 2440 3    60   Input ~ 0
-PD2
+PD4_ENC6
 Text GLabel 6790 2440 3    60   Input ~ 0
-PD3
-Text GLabel 4040 4410 2    60   Input ~ 0
-PD0
-Text GLabel 4040 4510 2    60   Input ~ 0
-PD1
-Text GLabel 4040 4610 2    60   Input ~ 0
-PD2
-Text GLabel 4040 4710 2    60   Input ~ 0
-PD3
+PD3_ENC7
 $Comp
 L AVR-ISP-10 CON?
@@
 	5490 2500 5490 2440
 Wire Wire Line
-	4960 2500 5310 2500
-Wire Wire Line
-	5310 2500 5490 2500
+	4960 2500 5490 2500
 Connection ~ 5310 2500
 Wire Wire Line
-	4960 2880 5310 2880
-Wire Wire Line
-	5310 2880 5590 2880
+	4960 2880 5590 2880
 Wire Wire Line
 	5310 2880 5310 2800
@@
 	6780 3610 6400 3610
 Wire Wire Line
-	6400 3510 6400 3610
-Wire Wire Line
-	6400 3610 6400 3710
-Wire Wire Line
-	6400 3710 6400 3810
+	6400 3510 6400 3810
 Connection ~ 6400 3610
 Connection ~ 6400 3710
@@
 	5750 3810 6150 3810
 Wire Wire Line
-	2020 1180 2020 1440
-Wire Wire Line
-	2020 1440 2020 1710
+	2020 1180 2020 1710
 Wire Wire Line
 	1640 1090 1640 1180
-Text GLabel 4040 4910 2    60   Input ~ 0
-PD5_encA
-Text GLabel 4040 2710 2    60   Input ~ 0
-PB1_encSW
 $Comp
 L Rotary_Encoder_Switch SW?
@@
 $EndComp
 Wire Wire Line
-	5250 4740 5590 4740
-Wire Wire Line
-	5590 4740 6190 4740
+	5250 4740 6190 4740
 Connection ~ 5590 4740
 $Comp
@@
 	5890 5040 5590 5040
 Text GLabel 5590 4440 0    60   Input ~ 0
-PD5_encA
+PA1_encA
 Text GLabel 5590 5040 0    60   Input ~ 0
-PD4_encB
+PA2_encB
 $Comp
 L C C?
@@
 $EndComp
 Text GLabel 7490 4640 2    60   Input ~ 0
-PB1_encSW
-Wire Wire Line
-	6790 4640 7280 4640
-Wire Wire Line
-	7280 4640 7490 4640
+PA3_encSW
+Wire Wire Line
+	6790 4640 7490 4640
 Wire Wire Line
 	7280 4940 6790 4940
@@
 $EndComp
 Wire Wire Line
-	8990 2250 8990 2520
-Wire Wire Line
-	8990 2520 8990 2810
-Wire Wire Line
-	8990 2810 8990 3080
-Wire Wire Line
-	8990 3080 8990 3220
+	8990 2250 8990 3220
 Connection ~ 8990 2520
 Connection ~ 8990 2810
@@
 $EndComp
 Text GLabel 7810 2880 0    60   Input ~ 0
-PB0_LED
-Text GLabel 4040 2610 2    60   Input ~ 0
-PB0_LED
+PC4_LED
 $Comp
 L R R?
@@
 $EndComp
 Wire Wire Line
-	8690 2250 8690 2520
-Wire Wire Line
-	8690 2520 8690 2810
-Wire Wire Line
-	8690 2810 8690 3080
+	8690 2250 8690 3080
 Connection ~ 8690 2520
 Connection ~ 8690 2810
@@
 $EndComp
 Wire Wire Line
-	2890 1060 2890 1240
-Wire Wire Line
-	2890 1240 2890 1410
+	2890 1060 2890 1410
 $Comp
 L +5V #PWR?
@@
 $EndComp
 Wire Wire Line
-	2990 5410 3040 5410
-Wire Wire Line
-	3040 5410 3090 5410
+	2990 5410 3090 5410
 Connection ~ 3040 5410
 $Comp
@@
 $EndComp
 Wire Wire Line
-	3190 1060 3190 1240
-Wire Wire Line
-	3190 1240 3190 1410
+	3190 1060 3190 1410
 $Comp
 L +5V #PWR?
@@
 $EndComp
 Wire Wire Line
-	1690 2910 1870 2910
-Wire Wire Line
-	1870 2910 2040 2910
+	1690 2910 2040 2910
 $Comp
 L +5V #PWR?
@@
 NoConn ~ 4040 4110
 NoConn ~ 4040 4010
-NoConn ~ 4040 3910
 NoConn ~ 4040 3810
-NoConn ~ 4040 3710
-NoConn ~ 4040 3610
-NoConn ~ 4040 3510
 NoConn ~ 4040 3010
 NoConn ~ 4040 2410
@@
 NoConn ~ 4040 2210
 NoConn ~ 4040 2110
-NoConn ~ 4040 2010
-NoConn ~ 4040 1910
-NoConn ~ 4040 1810
 NoConn ~ 4040 1710
 NoConn ~ 2040 2110
@@
 	1740 1440 2020 1440
 Connection ~ 2020 1440
-Text GLabel 4040 2810 2    60   Input ~ 0
-PB2_SW1
-Text GLabel 4040 2910 2    60   Input ~ 0
-PB3_SW2
 $Comp
 L SW_PUSH SW?
@@
 	9240 4740 9240 5010
 Text GLabel 9240 4000 2    60   Input ~ 0
-PB2_SW1
+PC1_SW1
 Text GLabel 9240 5010 2    60   Input ~ 0
-PB3_SW2
+PC2_SW2
 $Comp
 L SW_PUSH SW?
@@
 	1    0    0    -1
 $EndComp
+Text GLabel 4040 2010 2    60   Input ~ 0
+PA3_encSW
+Text GLabel 4040 1810 2    60   Input ~ 0
+PA1_encA
+Text GLabel 4040 1910 2    60   Input ~ 0
+PA2_encB
+Text GLabel 4040 3910 2    60   Input ~ 0
+PC4_LED
+Text GLabel 4040 3610 2    60   Input ~ 0
+PC1_SW1
+Text GLabel 4040 3710 2    60   Input ~ 0
+PC2_SW2
+Text GLabel 4040 5010 2    60   Input ~ 0
+PD6_ENC4
+Text GLabel 4040 4910 2    60   Input ~ 0
+PD5_ENC5
 Text GLabel 4040 4810 2    60   Input ~ 0
-PD4_encB
+PD4_ENC6
+Text GLabel 4040 4710 2    60   Input ~ 0
+PD3_ENC7
+Text GLabel 4040 3510 2    60   Input ~ 0
+PC0_RS
+NoConn ~ 4040 2610
+NoConn ~ 4040 2710
+NoConn ~ 4040 2810
+NoConn ~ 4040 2910
+NoConn ~ 4040 4410
+NoConn ~ 4040 4510
+NoConn ~ 4040 4610
 $EndSCHEMATC

Commit message: morse-torch v2 initial commit
Parts:
- C? (x9): symbol C -> device:C
- CON?: symbol AVR-ISP-10 -> atmel:AVR-ISP-10
- D? (x4): symbol LED -> device:LED
- DS?: symbol LCD8X2 -> latarka_1-rescue:LCD8X2
- Q?: symbol 2N2219 -> transistors:2N2219
- R? (x8): symbol R -> device:R
- RV?: symbol POT -> device:POT
- SW? (x4): symbol SW_PUSH -> latarka_1-rescue:SW_PUSH
- SW?: symbol Rotary_Encoder_Switch -> device:Rotary_Encoder_Switch
- U?: symbol ATMEGA32-16PU -> atmel:ATMEGA32-16PU
