File: v_2/KiCad/morse-torch_v2/morse-torch_v2.sch (KiCad schematic (older format))
At the start: 42 parts

Commit message: started pcb design, step-up converter needs approval
Parts:
- removed C? (x2): 4,7uF, symbol Device:C
- removed D?: D_Schottky, symbol Device:D_Schottky
- removed L?: 3,3uH, symbol Device:L
- removed R1: 390k, symbol Device:R
- removed R2: 130k, symbol Device:R
- removed U?: LM27313XMF, Package_TO_SOT_SMD:SOT-23-5, symbol Regulator_Switching:LM27313XMF
- added C1, C2, C3: 100nF, symbol Device:C
- added C18, C21: 100n, Capacitor_SMD:C_0805_2012Metric_Pad1.15x1.40mm_HandSolder, symbol Device:C
- added C19, C22: 100u, Capacitor_SMD:CP_Elec_6.3x5.4, symbol Device:CP
- added C20: 470p, Capacitor_SMD:C_0805_2012Metric_Pad1.15x1.40mm_HandSolder, symbol Device:C
- added C4, C5: 22pF, Capacitor_SMD:C_0805_2012Metric_Pad1.15x1.40mm_HandSolder, symbol Device:C
- added D1, D2, D3: BAT54C, Package_TO_SOT_SMD:SOT-23, symbol Diode:BAT54C
- added D12: MBR0520, Diode_SMD:D_SOD-123, symbol Diode:MBR0520
- added J6: BATT, Connector_PinHeader_2.54mm:PinHeader_1x02_P2.54mm_Vertical, symbol Connector_Generic:Conn_01x02
- added J7: PWR, Connector_PinHeader_2.54mm:PinHeader_1x02_P2.54mm_Vertical, symbol Connector_Generic:Conn_01x02
- added L1: 10uH, symbol Device:L
- added L4: 10u, Inductor_THT:L_Radial_D6.0mm_P4.00mm, symbol Device:L
- added R11: 1, Resistor_SMD:R_0805_2012Metric_Pad1.15x1.40mm_HandSolder, symbol Device:R
- added R12: 33k, Resistor_SMD:R_0805_2012Metric_Pad1.15x1.40mm_HandSolder, symbol Device:R
- added R13, R14: 100k, Resistor_SMD:R_0805_2012Metric_Pad1.15x1.40mm_HandSolder, symbol Device:R
- added R3: 10k, symbol Device:R
- added U1: ATmega328P-AU, Package_QFP:TQFP-32_7x7mm_P0.8mm, symbol MCU_Microchip_ATmega:ATmega328P-AU
- added U5: MC34063AD, Package_SO:SOIC-8_3.9x4.9mm_P1.27mm, symbol Regulator_Switching:MC34063AD
- added Y1: Crystal, Crystal:Crystal_HC49-U_Vertical, symbol Device:Crystal
- J2, J3: renamed from J?; footprint (none) -> Connector_PinHeader_2.54mm:PinHeader_1x04_P2.54mm_Vertical
- J4: renamed from J?; footprint (none) -> Connector_PinHeader_2.54mm:PinHeader_2x03_P2.54mm_Vertical
- J5: renamed from J?; footprint (none) -> Connector_PinHeader_2.54mm:PinHeader_1x02_P2.54mm_Vertical
- RV1: renamed from RV?; footprint (none) -> Potentiometer_THT:Potentiometer_Piher_PT-6-V_Vertical
- SW1, SW2: renamed from SW?; footprint (none) -> Button_Switch_THT:SW_PUSH_6mm
- SW3: renamed from SW?; footprint (none) -> Rotary_Encoder:RotaryEncoder_Alps_EC11E-Switch_Vertical_H20mm
- U4: renamed from U?; footprint Display:NHD-0420H1Z -> Connector_PinHeader_2.54mm:PinHeader_2x07_P2.54mm_Vertical
- gave numbers to parts that had none: 26
Connections:
- net +5V: now also C2.1, J7.1 (Pin_1), L1.1, R3.1, U1.18 (AVCC), U1.4 (VCC), U1.6 (VCC)
- net BUTTON_1: now also D1.1, U1.12 (PB0)
- net BUTTON_2: now also D1.2, U1.13 (PB1)
- net ENC_A: now also D2.2, U1.14 (PB2)
- net ENC_B: now also D2.1, U1.22 (ADC7)
- net ENC_BUTTON: now also D3.1, U1.19 (ADC6)
- net GND: now also C1.1, C18.2, C19.1, C2.2, C20.2, C21.2, C22.1, C3.2, C4.2, C5.2, J6.2 (Pin_2), R12.1, U1.21 (GND), U1.3 (GND), U1.5 (GND), U5.2 (SwE), U5.4 (GND)
- net LCD_DATA4: now also U1.2 (PD4)
- net LCD_DATA5: now also U1.9 (PD5)
- net LCD_DATA6: now also U1.10 (PD6)
- net LCD_DATA7: now also U1.11 (PD7)
- net LCD_E: now also U1.25 (PC2)
- net LCD_RS: now also U1.26 (PC3)
- net LIGHT_SW: now also U1.24 (PC1)
- net MISO: now also U1.16 (PB4)
- net MOSI: now also U1.15 (PB3)
- net RESET: now also R3.2, U1.29 (~RESET~/PC6)
- net RXD: now also U1.30 (PD0)
- net SCK: now also U1.17 (PB5)
- net SCL: now also U1.28 (PC5)
- net SDA: now also U1.27 (PC4)
- net TXD: now also U1.31 (PD1)
- net VCC: now also C18.1, C19.2, J6.1 (Pin_1), R11.2, U1.23 (PC0), U5.6 (Vin)
- new net: C1.2, U1.20 (AREF)
- new net: D1.3, D2.3, D3.3, U1.32 (PD2)
- new net: C3.1, L1.2
- new net: D12.2 (A), L4.2, U5.1 (SwC)
- new net: C20.1, U5.3 (TC)
- new net: R12.2, R14.1, U5.5 (Vfb)
- new net: L4.1, R11.1, R13.1, U5.7 (Ipk)
- new net: R13.2, U5.8 (DC)
- new net 5V-converter: C21.1, C22.2, D12.1 (K), J7.2 (Pin_2), R14.2
- new net XTAL1: C4.1, U1.7 (XTAL1/PB6), Y1.1
- new net XTAL2: C5.1, U1.8 (XTAL2/PB7), Y1.2
- no-connect marks 2 -> 3

Commit message: changed uc to atmega32, added jtag interface, roughly set up final layout
Parts:
- removed C10, C11, C9: 100nF, symbol Device:C
- removed C18, C21: 100n, Capacitor_SMD:C_0805_2012Metric_Pad1.15x1.40mm_HandSolder, symbol Device:C
- removed C19, C22: 100u, Capacitor_SMD:CP_Elec_6.3x5.4, symbol Device:CP
- removed C20: 470p, Capacitor_SMD:C_0805_2012Metric_Pad1.15x1.40mm_HandSolder, symbol Device:C
- removed C6, C7: 22pF, symbol Device:C
- removed D10, D6, D7, D8, D9: D_Schottky, symbol Device:D_Schottky
- removed D12: MBR0520, Diode_SMD:D_SOD-123, symbol Diode:MBR0520
- removed L2: 10uH, symbol Device:L
- removed L4: 10u, Inductor_THT:L_Radial_D6.0mm_P4.00mm, symbol Device:L
- removed R10, R4: 10k, symbol Device:R
- removed R11: 1, Resistor_SMD:R_0805_2012Metric_Pad1.15x1.40mm_HandSolder, symbol Device:R
- removed R12: 33k, Resistor_SMD:R_0805_2012Metric_Pad1.15x1.40mm_HandSolder, symbol Device:R
- removed R13, R14: 100k, Resistor_SMD:R_0805_2012Metric_Pad1.15x1.40mm_HandSolder, symbol Device:R
- removed U2: ATmega32-16AU, Package_QFP:TQFP-44_10x10mm_P0.8mm, symbol MCU_Microchip_ATmega:ATmega32-16AU
- removed U5: MC34063AD, Package_SO:SOIC-8_3.9x4.9mm_P1.27mm, symbol Regulator_Switching:MC34063AD
- removed Y2: Crystal, symbol Device:Crystal
- added C1, C3: 100n, Capacitor_SMD:C_0805_2012Metric_Pad1.15x1.40mm_HandSolder, symbol Device:C
- added C2, C4: 100u, Capacitor_SMD:CP_Elec_6.3x5.4, symbol Device:CP
- added Ct: 470p, Capacitor_SMD:C_0805_2012Metric_Pad1.15x1.40mm_HandSolder, symbol Device:C
- added D1: MBR0520, Diode_SMD:D_SOD-123, symbol Diode:MBR0520
- added L1: 82u, Inductor_THT:L_Radial_D6.0mm_P4.00mm, symbol Device:L
- added Q2: BC817, Package_TO_SOT_SMD:SOT-23, symbol Transistor_BJT:BC817
- added R1: 130k, Resistor_SMD:R_0805_2012Metric_Pad1.15x1.40mm_HandSolder, symbol Device:R
- added R2: 390k, Resistor_SMD:R_0805_2012Metric_Pad1.15x1.40mm_HandSolder, symbol Device:R
- added R3: 100k, Resistor_SMD:R_0805_2012Metric_Pad1.15x1.40mm_HandSolder, symbol Device:R
- added R?, Rsw, Rsw2, Rtr: 10k, symbol Device:R
- added Rsc: 1, Resistor_SMD:R_0805_2012Metric_Pad1.15x1.40mm_HandSolder, symbol Device:R
- added U?: MC34063AD, Package_SO:SOIC-8_3.9x4.9mm_P1.27mm, symbol Regulator_Switching:MC34063AD
- added U?: 24LC128, symbol Memory_EEPROM:24LC128
- C1, C2, C3: footprint (none) -> Capacitor_SMD:C_0805_2012Metric_Pad1.15x1.40mm_HandSolder
- L1: footprint (none) -> Inductor_SMD:L_0805_2012Metric_Pad1.15x1.40mm_HandSolder
- R3: footprint (none) -> Resistor_SMD:R_0805_2012Metric_Pad1.15x1.40mm_HandSolder
Connections:
- net 5V-converter is gone; now on net VCC: J7.2 (Pin_2)
- net +5V: now also U?.8 (VCC); no longer J7.1 (Pin_1), Q1.3 (C)
- net GND: now also Q1.2 (E), C1.2, C2.1, C3.2, C4.1, Ct.2, Q2.2 (E), R1.1, U?.2 (SwE), U?.4 (GND), U?.4 (GND); no longer J5.2 (Pin_2)
- net LIGHT_SW: now also Rtr.2
- net SCL: now also U?.6 (SCL)
- net SDA: now also U?.5 (SDA)
- net VCC: now also J5.2 (Pin_2)
- net write-protection: now reaches U1.1 (PD3)
- net write-protection: now also R?.2, U?.7 (WP)
- net at Q1.1 (B): now also Rtr.1
- net LCD_DATA0: no longer names the net of U4.7 (DB0)
- net LCD_DATA1: no longer names the net of U4.8 (DB1)
- net LCD_DATA2: no longer names the net of U4.9 (DB2)
- net LCD_DATA3: no longer names the net of U4.10 (DB3)
- net LIGHT_VCC: no longer names the net of J5.1 (Pin_1)
- net LIGHT_VCC: now also Q2.3 (C), Rsw.2; no longer Q1.2 (E)
- new net: C1.1, C2.2, J7.1 (Pin_1), Rsc.2, U?.6 (Vin)
- new net: D1.2 (A), L1.2, U?.1 (SwC)
- new net: Ct.1, U?.3 (TC)
- new net: R1.2, R2.1, U?.5 (Vfb)
- new net: L1.1, R3.1, Rsc.1, U?.7 (Ipk)
- new net: R3.2, U?.8 (DC)
- new net: Q1.3 (C), Rsw.1, Rsw2.1
- new net: Q2.1 (B), Rsw2.2
- new net +5C: R?.1
- new net Uout=+5V: C3.1, C4.2, D1.1 (K), R2.2
- no-connect marks 3 -> 10
Other:
- moved on the sheet: C1, C12, C14, C15, C17, C2, C3, C4, C5, C8, D1, D2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
